Commit message: correct orientation of Base mesh

File: ur_description/urdf/ur10.urdf.xacro (robot description, xacro)
@@ -48,5 +48,5 @@
 		    <mesh filename="package://ur_description/meshes/ur10/visual/Base.stl" />
 		  </geometry>
-		  <origin xyz="0.0 0.0 0.003" rpy="0.0 0.0 ${3.0 * pi / 4.0}" />
+		  <origin xyz="0.0 0.0 0.003" rpy="0.0 0.0 0.0" />
 		  <material name="UR/Blue" />
 		</visual>
@@ -55,5 +55,5 @@
 		    <mesh filename="package://ur_description/meshes/ur10/collision/Base.stl" />
 		  </geometry>
-		  <origin xyz="0.0 0.0 0.003" rpy="0.0 0.0 ${3.0 * pi / 4.0}" />
+		  <origin xyz="0.0 0.0 0.003" rpy="0.0 0.0 0.0" />
 		</collision>
 		<inertial>

Commit message: updates from ros-industrial

File: ur_description/urdf/ur10.urdf.xacro (robot description, xacro)
@@ -5,6 +5,6 @@
   Contributers: Jimmy Da Silva, Ajit Krisshna N L, Muhammad Asif Rana
 -->
-  <xacro:include filename="$(find ur_description)/urdf/ur10.transmission.xacro" />
-  <xacro:include filename="$(find ur_description)/urdf/ur10.gazebo.xacro" />
+  <xacro:include filename="$(find ur_description)/urdf/ur.transmission.xacro" />
+  <xacro:include filename="$(find ur_description)/urdf/ur.gazebo.xacro" />
   <property name="pi" value="3.14159265" />
   <!-- Inertia parameters -->
@@ -57,5 +57,5 @@
       <visual>
         <geometry>
-          <mesh filename="package://ur_description/meshes/ur10/visual/Base.dae"/>
+          <mesh filename="package://ur_description/meshes/ur10/visual/base.dae"/>
         </geometry>
         <material name="LightGrey">
@@ -88,5 +88,5 @@
       <visual>
         <geometry>
-          <mesh filename="package://ur_description/meshes/ur10/visual/Shoulder.dae"/>
+          <mesh filename="package://ur_description/meshes/ur10/visual/shoulder.dae"/>
         </geometry>
         <material name="LightGrey">
@@ -119,13 +119,13 @@
       <visual>
         <geometry>
-          <mesh filename="package://ur_description/meshes/ur10/visual/UpperArm.dae"/>
-        </geometry>
-        <material name="LightGrey">
-          <color rgba="0.7 0.7 0.7 1.0"/>
-        </material>
-      </visual>
-      <collision>
-        <geometry>
-          <mesh filename="package://ur_description/meshes/ur10/collision/upper_arm.stl"/>
+          <mesh filename="package://ur_description/meshes/ur10/visual/upperarm.dae"/>
+        </geometry>
+        <material name="LightGrey">
+          <color rgba="0.7 0.7 0.7 1.0"/>
+        </material>
+      </visual>
+      <collision>
+        <geometry>
+          <mesh filename="package://ur_description/meshes/ur10/collision/upperarm.stl"/>
         </geometry>
       </collision>
@@ -150,5 +150,5 @@
       <visual>
          <geometry>
-          <mesh filename="package://ur_description/meshes/ur10/visual/Forearm.dae"/>
+          <mesh filename="package://ur_description/meshes/ur10/visual/forearm.dae"/>
         </geometry>
         <material name="LightGrey">
@@ -181,13 +181,13 @@
       <visual>
         <geometry>
-          <mesh filename="package://ur_description/meshes/ur10/visual/Wrist1.dae"/>
-        </geometry>
-        <material name="LightGrey">
-          <color rgba="0.7 0.7 0.7 1.0"/>
-        </material>
-      </visual>
-      <collision>
-        <geometry>
-          <mesh filename="package://ur_description/meshes/ur10/collision/wrist_1.stl"/>
+          <mesh filename="package://ur_description/meshes/ur10/visual/wrist1.dae"/>
+        </geometry>
+        <material name="LightGrey">
+          <color rgba="0.7 0.7 0.7 1.0"/>
+        </material>
+      </visual>
+      <collision>
+        <geometry>
+          <mesh filename="package://ur_description/meshes/ur10/collision/wrist1.stl"/>
         </geometry>
       </collision>
@@ -212,13 +212,13 @@
       <visual>
         <geometry>
-          <mesh filename="package://ur_description/meshes/ur10/visual/Wrist2.dae"/>
-        </geometry>
-        <material name="LightGrey">
-          <color rgba="0.7 0.7 0.7 1.0"/>
-        </material>
-      </visual>
-      <collision>
-        <geometry>
-          <mesh filename="package://ur_description/meshes/ur10/collision/wrist_2.stl"/>
+          <mesh filename="package://ur_description/meshes/ur10/visual/wrist2.dae"/>
+        </geometry>
+        <material name="LightGrey">
+          <color rgba="0.7 0.7 0.7 1.0"/>
+        </material>
+      </visual>
+      <collision>
+        <geometry>
+          <mesh filename="package://ur_description/meshes/ur10/collision/wrist2.stl"/>
         </geometry>
       </collision>
@@ -243,13 +243,13 @@
       <visual>
         <geometry>
-          <mesh filename="package://ur_description/meshes/ur10/visual/Wrist3.dae"/>
-        </geometry>
-        <material name="LightGrey">
-          <color rgba="0.7 0.7 0.7 1.0"/>
-        </material>
-      </visual>
-      <collision>
-        <geometry>
-          <mesh filename="package://ur_description/meshes/ur10/collision/wrist_3.stl"/>
+          <mesh filename="package://ur_description/meshes/ur10/visual/wrist3.dae"/>
+        </geometry>
+        <material name="LightGrey">
+          <color rgba="0.7 0.7 0.7 1.0"/>
+        </material>
+      </visual>
+      <collision>
+        <geometry>
+          <mesh filename="package://ur_description/meshes/ur10/collision/wrist3.stl"/>
         </geometry>
       </collision>
@@ -271,6 +271,24 @@
       </collision>
     </link>
-    <xacro:ur10_arm_transmission prefix="${prefix}" />
-    <xacro:ur10_arm_gazebo prefix="${prefix}" />
+    <xacro:ur_arm_transmission prefix="${prefix}" />
+    <xacro:ur_arm_gazebo prefix="${prefix}" />
+    <!-- ROS base_link to UR 'Base' Coordinates transform -->
+    <link name="${prefix}base"/>
+    <joint name="${prefix}base_link-base_fixed_joint" type="fixed">
+      <!-- NOTE: this rotation is only needed as long as base_link itself is
+                 not corrected wrt the real robot (ie: rotated over 180
+                 degrees)
+      -->
+      <origin xyz="0 0 0" rpy="0 0 ${-pi}"/>
+      <parent link="${prefix}base_link"/>
+      <child link="${prefix}base"/>
+    </joint>
+    <!-- Frame coincident with all-zeros TCP on UR controller -->
+    <link name="${prefix}tool0"/>
+    <joint name="${prefix}wrist_3_link-tool0_fixed_joint" type="fixed">
+      <origin xyz="0 ${wrist_3_length} 0" rpy="${pi/-2.0} 0 0"/>
+      <parent link="${prefix}wrist_3_link"/>
+      <child link="${prefix}tool0"/>
+    </joint>
   </xacro:macro>
 </robot>
